Commit message: ready to generate data from server

File: assets/urdf/1be987c137d37f0b7c15f7bdb6fa82dd/1be987c137d37f0b7c15f7bdb6fa82dd.urdf (robot description, URDF)
Before this commit: robot 1be987c137d37f0b7c15f7bdb6fa82dd, 1 links, 0 joints
Links:
- link 1be987c137d37f0b7c15f7bdb6fa82dd: geometry collision mesh filename=/home/jongsoo/catkin_ws/src/stable_push_data_check/assets/u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 scale=1 1 1; visual mesh filename=/home/jongsoo/catkin_ws/src/stable_push_data_check/assets/u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 scale=1 1 1

File: assets/urdf/1be987c137d37f0b7c15f7bdb6fa82dd_0/1be987c137d37f0b7c15f7bdb6fa82dd_0.urdf (robot description, URDF)
Before this commit: robot 1be987c137d37f0b7c15f7bdb6fa82dd_0, 1 links, 0 joints
Links:
- link 1be987c137d37f0b7c15f7bdb6fa82dd_0: geometry collision mesh filename=/home/jongsoo/catkin_ws/src/stable_push_data_check/assets/u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 scale=1 1 1; visual mesh filename=/home/jongsoo/catkin_ws/src/stable_push_data_check/assets/u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 scale=1 1 1

File: assets/urdf/1be987c137d37f0b7c15f7bdb6fa82dd_1/1be987c137d37f0b7c15f7bdb6fa82dd_1.urdf (robot description, URDF)
Before this commit: robot 1be987c137d37f0b7c15f7bdb6fa82dd_1, 1 links, 0 joints
Links:
- link 1be987c137d37f0b7c15f7bdb6fa82dd_1: geometry collision mesh filename=/home/jongsoo/catkin_ws/src/stable_push_data_check/assets/u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 scale=1 1 1; visual mesh filename=/home/jongsoo/catkin_ws/src/stable_push_data_check/assets/u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 scale=1 1 1

File: assets/urdf/1be987c137d37f0b7c15f7bdb6fa82dd_2/1be987c137d37f0b7c15f7bdb6fa82dd_2.urdf (robot description, URDF)
Before this commit: robot 1be987c137d37f0b7c15f7bdb6fa82dd_2, 1 links, 0 joints
Links:
- link 1be987c137d37f0b7c15f7bdb6fa82dd_2: geometry collision mesh filename=/home/jongsoo/catkin_ws/src/stable_push_data_check/assets/u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 scale=1 1 1; visual mesh filename=/home/jongsoo/catkin_ws/src/stable_push_data_check/assets/u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 scale=1 1 1

File: assets/urdf/1be987c137d37f0b7c15f7bdb6fa82dd_3/1be987c137d37f0b7c15f7bdb6fa82dd_3.urdf (robot description, URDF)
Before this commit: robot 1be987c137d37f0b7c15f7bdb6fa82dd_3, 1 links, 0 joints
Links:
- link 1be987c137d37f0b7c15f7bdb6fa82dd_3: geometry collision mesh filename=/home/jongsoo/catkin_ws/src/stable_push_data_check/assets/u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 scale=1 1 1; visual mesh filename=/home/jongsoo/catkin_ws/src/stable_push_data_check/assets/u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 scale=1 1 1

File: assets/urdf/1be987c137d37f0b7c15f7bdb6fa82dd_4/1be987c137d37f0b7c15f7bdb6fa82dd_4.urdf (robot description, URDF)
Before this commit: robot 1be987c137d37f0b7c15f7bdb6fa82dd_4, 1 links, 0 joints
Links:
- link 1be987c137d37f0b7c15f7bdb6fa82dd_4: geometry collision mesh filename=/home/jongsoo/catkin_ws/src/stable_push_data_check/assets/u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 scale=1 1 1; visual mesh filename=/home/jongsoo/catkin_ws/src/stable_push_data_check/assets/u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 scale=1 1 1

File: assets/urdf/1be987c137d37f0b7c15f7bdb6fa82dd_5/1be987c137d37f0b7c15f7bdb6fa82dd_5.urdf (robot description, URDF)
Before this commit: robot 1be987c137d37f0b7c15f7bdb6fa82dd_5, 1 links, 0 joints
Links:
- link 1be987c137d37f0b7c15f7bdb6fa82dd_5: geometry collision mesh filename=/home/jongsoo/catkin_ws/src/stable_push_data_check/assets/u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 scale=1 1 1; visual mesh filename=/home/jongsoo/catkin_ws/src/stable_push_data_check/assets/u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 scale=1 1 1

File: assets/urdf/1be987c137d37f0b7c15f7bdb6fa82dd_6/1be987c137d37f0b7c15f7bdb6fa82dd_6.urdf (robot description, URDF)
Before this commit: robot 1be987c137d37f0b7c15f7bdb6fa82dd_6, 1 links, 0 joints
Links:
- link 1be987c137d37f0b7c15f7bdb6fa82dd_6: geometry collision mesh filename=/home/jongsoo/catkin_ws/src/stable_push_data_check/assets/u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 scale=1 1 1; visual mesh filename=/home/jongsoo/catkin_ws/src/stable_push_data_check/assets/u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 scale=1 1 1

File: assets/urdf/1be987c137d37f0b7c15f7bdb6fa82dd_7/1be987c137d37f0b7c15f7bdb6fa82dd_7.urdf (robot description, URDF)
Before this commit: robot 1be987c137d37f0b7c15f7bdb6fa82dd_7, 1 links, 0 joints
Links:
- link 1be987c137d37f0b7c15f7bdb6fa82dd_7: geometry collision mesh filename=/home/jongsoo/catkin_ws/src/stable_push_data_check/assets/u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 scale=1 1 1; visual mesh filename=/home/jongsoo/catkin_ws/src/stable_push_data_check/assets/u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 scale=1 1 1

File: assets/urdf/1be987c137d37f0b7c15f7bdb6fa82dd_8/1be987c137d37f0b7c15f7bdb6fa82dd_8.urdf (robot description, URDF)
Before this commit: robot 1be987c137d37f0b7c15f7bdb6fa82dd_8, 1 links, 0 joints
Links:
- link 1be987c137d37f0b7c15f7bdb6fa82dd_8: geometry collision mesh filename=/home/jongsoo/catkin_ws/src/stable_push_data_check/assets/u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 scale=1 1 1; visual mesh filename=/home/jongsoo/catkin_ws/src/stable_push_data_check/assets/u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 scale=1 1 1

File: assets/urdf/1be987c137d37f0b7c15f7bdb6fa82dd_9/1be987c137d37f0b7c15f7bdb6fa82dd_9.urdf (robot description, URDF)
Before this commit: robot 1be987c137d37f0b7c15f7bdb6fa82dd_9, 1 links, 0 joints
Links:
- link 1be987c137d37f0b7c15f7bdb6fa82dd_9: geometry collision mesh filename=/home/jongsoo/catkin_ws/src/stable_push_data_check/assets/u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 scale=1 1 1; visual mesh filename=/home/jongsoo/catkin_ws/src/stable_push_data_check/assets/u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 scale=1 1 1

File: assets/urdf/2eb4cfc59205bb3a147c505998f546dd/2eb4cfc59205bb3a147c505998f546dd.urdf (robot description, URDF)
Before this commit: robot 2eb4cfc59205bb3a147c505998f546dd, 1 links, 0 joints
Links:
- link 2eb4cfc59205bb3a147c505998f546dd: geometry collision mesh filename=/home/jongsoo/catkin_ws/src/stable_push_data_check/assets/u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 scale=1 1 1; visual mesh filename=/home/jongsoo/catkin_ws/src/stable_push_data_check/assets/u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 scale=1 1 1

File: assets/urdf/2eb4cfc59205bb3a147c505998f546dd_0/2eb4cfc59205bb3a147c505998f546dd_0.urdf (robot description, URDF)
Before this commit: robot 2eb4cfc59205bb3a147c505998f546dd_0, 1 links, 0 joints
Links:
- link 2eb4cfc59205bb3a147c505998f546dd_0: geometry collision mesh filename=/home/jongsoo/catkin_ws/src/stable_push_data_check/assets/u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 scale=1 1 1; visual mesh filename=/home/jongsoo/catkin_ws/src/stable_push_data_check/assets/u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 scale=1 1 1

File: assets/urdf/2eb4cfc59205bb3a147c505998f546dd_1/2eb4cfc59205bb3a147c505998f546dd_1.urdf (robot description, URDF)
Before this commit: robot 2eb4cfc59205bb3a147c505998f546dd_1, 1 links, 0 joints
Links:
- link 2eb4cfc59205bb3a147c505998f546dd_1: geometry collision mesh filename=/home/jongsoo/catkin_ws/src/stable_push_data_check/assets/u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 scale=1 1 1; visual mesh filename=/home/jongsoo/catkin_ws/src/stable_push_data_check/assets/u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 scale=1 1 1

File: assets/urdf/2eb4cfc59205bb3a147c505998f546dd_2/2eb4cfc59205bb3a147c505998f546dd_2.urdf (robot description, URDF)
Before this commit: robot 2eb4cfc59205bb3a147c505998f546dd_2, 1 links, 0 joints
Links:
- link 2eb4cfc59205bb3a147c505998f546dd_2: geometry collision mesh filename=/home/jongsoo/catkin_ws/src/stable_push_data_check/assets/u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 scale=1 1 1; visual mesh filename=/home/jongsoo/catkin_ws/src/stable_push_data_check/assets/u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 scale=1 1 1

File: assets/urdf/2eb4cfc59205bb3a147c505998f546dd_3/2eb4cfc59205bb3a147c505998f546dd_3.urdf (robot description, URDF)
Before this commit: robot 2eb4cfc59205bb3a147c505998f546dd_3, 1 links, 0 joints
Links:
- link 2eb4cfc59205bb3a147c505998f546dd_3: geometry collision mesh filename=/home/jongsoo/catkin_ws/src/stable_push_data_check/assets/u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 scale=1 1 1; visual mesh filename=/home/jongsoo/catkin_ws/src/stable_push_data_check/assets/u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 scale=1 1 1

File: assets/urdf/2eb4cfc59205bb3a147c505998f546dd_4/2eb4cfc59205bb3a147c505998f546dd_4.urdf (robot description, URDF)
Before this commit: robot 2eb4cfc59205bb3a147c505998f546dd_4, 1 links, 0 joints
Links:
- link 2eb4cfc59205bb3a147c505998f546dd_4: geometry collision mesh filename=/home/jongsoo/catkin_ws/src/stable_push_data_check/assets/u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 scale=1 1 1; visual mesh filename=/home/jongsoo/catkin_ws/src/stable_push_data_check/assets/u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 scale=1 1 1

File: assets/urdf/2eb4cfc59205bb3a147c505998f546dd_5/2eb4cfc59205bb3a147c505998f546dd_5.urdf (robot description, URDF)
Before this commit: robot 2eb4cfc59205bb3a147c505998f546dd_5, 1 links, 0 joints
Links:
- link 2eb4cfc59205bb3a147c505998f546dd_5: geometry collision mesh filename=/home/jongsoo/catkin_ws/src/stable_push_data_check/assets/u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 scale=1 1 1; visual mesh filename=/home/jongsoo/catkin_ws/src/stable_push_data_check/assets/u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 scale=1 1 1

File: assets/urdf/2eb4cfc59205bb3a147c505998f546dd_6/2eb4cfc59205bb3a147c505998f546dd_6.urdf (robot description, URDF)
Before this commit: robot 2eb4cfc59205bb3a147c505998f546dd_6, 1 links, 0 joints
Links:
- link 2eb4cfc59205bb3a147c505998f546dd_6: geometry collision mesh filename=/home/jongsoo/catkin_ws/src/stable_push_data_check/assets/u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 scale=1 1 1; visual mesh filename=/home/jongsoo/catkin_ws/src/stable_push_data_check/assets/u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 scale=1 1 1

File: assets/urdf/2eb4cfc59205bb3a147c505998f546dd_7/2eb4cfc59205bb3a147c505998f546dd_7.urdf (robot description, URDF)
Before this commit: robot 2eb4cfc59205bb3a147c505998f546dd_7, 1 links, 0 joints
Links:
- link 2eb4cfc59205bb3a147c505998f546dd_7: geometry collision mesh filename=/home/jongsoo/catkin_ws/src/stable_push_data_check/assets/u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 scale=1 1 1; visual mesh filename=/home/jongsoo/catkin_ws/src/stable_push_data_check/assets/u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 scale=1 1 1
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
Commit message: add data augment and status

File: assets/urdf/1be987c137d37f0b7c15f7bdb6fa82dd/1be987c137d37f0b7c15f7bdb6fa82dd.urdf (robot description, URDF)
Before this commit: robot 1be987c137d37f0b7c15f7bdb6fa82dd, 1 links, 0 joints
Links:
- link 1be987c137d37f0b7c15f7bdb6fa82dd: geometry collision mesh filename=/home/rise/catkin_ws/src/stable_push_data_gen/assets/urdf/1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 scale=1 1 1; visual mesh filename=/home/rise/catkin_ws/src/stable_push_data_gen/assets/urdf/1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 scale=1 1 1

File: assets/urdf/1be987c137d37f0b7c15f7bdb6fa82dd_0/1be987c137d37f0b7c15f7bdb6fa82dd_0.urdf (robot description, URDF)
Before this commit: robot 1be987c137d37f0b7c15f7bdb6fa82dd_0, 1 links, 0 joints
Links:
- link 1be987c137d37f0b7c15f7bdb6fa82dd_0: geometry collision mesh filename=/home/rise/catkin_ws/src/stable_push_data_gen/assets/urdf/1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 scale=1 1 1; visual mesh filename=/home/rise/catkin_ws/src/stable_push_data_gen/assets/urdf/1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 scale=1 1 1

File: assets/urdf/1be987c137d37f0b7c15f7bdb6fa82dd_1/1be987c137d37f0b7c15f7bdb6fa82dd_1.urdf (robot description, URDF)
Before this commit: robot 1be987c137d37f0b7c15f7bdb6fa82dd_1, 1 links, 0 joints
Links:
- link 1be987c137d37f0b7c15f7bdb6fa82dd_1: geometry collision mesh filename=/home/rise/catkin_ws/src/stable_push_data_gen/assets/urdf/1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 scale=1 1 1; visual mesh filename=/home/rise/catkin_ws/src/stable_push_data_gen/assets/urdf/1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 scale=1 1 1

File: assets/urdf/1be987c137d37f0b7c15f7bdb6fa82dd_2/1be987c137d37f0b7c15f7bdb6fa82dd_2.urdf (robot description, URDF)
Before this commit: robot 1be987c137d37f0b7c15f7bdb6fa82dd_2, 1 links, 0 joints
Links:
- link 1be987c137d37f0b7c15f7bdb6fa82dd_2: geometry collision mesh filename=/home/rise/catkin_ws/src/stable_push_data_gen/assets/urdf/1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 scale=1 1 1; visual mesh filename=/home/rise/catkin_ws/src/stable_push_data_gen/assets/urdf/1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 scale=1 1 1

File: assets/urdf/1be987c137d37f0b7c15f7bdb6fa82dd_3/1be987c137d37f0b7c15f7bdb6fa82dd_3.urdf (robot description, URDF)
Before this commit: robot 1be987c137d37f0b7c15f7bdb6fa82dd_3, 1 links, 0 joints
Links:
- link 1be987c137d37f0b7c15f7bdb6fa82dd_3: geometry collision mesh filename=/home/rise/catkin_ws/src/stable_push_data_gen/assets/urdf/1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 scale=1 1 1; visual mesh filename=/home/rise/catkin_ws/src/stable_push_data_gen/assets/urdf/1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 scale=1 1 1

File: assets/urdf/1be987c137d37f0b7c15f7bdb6fa82dd_4/1be987c137d37f0b7c15f7bdb6fa82dd_4.urdf (robot description, URDF)
Before this commit: robot 1be987c137d37f0b7c15f7bdb6fa82dd_4, 1 links, 0 joints
Links:
- link 1be987c137d37f0b7c15f7bdb6fa82dd_4: geometry collision mesh filename=/home/rise/catkin_ws/src/stable_push_data_gen/assets/urdf/1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 scale=1 1 1; visual mesh filename=/home/rise/catkin_ws/src/stable_push_data_gen/assets/urdf/1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 scale=1 1 1

File: assets/urdf/1be987c137d37f0b7c15f7bdb6fa82dd_5/1be987c137d37f0b7c15f7bdb6fa82dd_5.urdf (robot description, URDF)
Before this commit: robot 1be987c137d37f0b7c15f7bdb6fa82dd_5, 1 links, 0 joints
Links:
- link 1be987c137d37f0b7c15f7bdb6fa82dd_5: geometry collision mesh filename=/home/rise/catkin_ws/src/stable_push_data_gen/assets/urdf/1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 scale=1 1 1; visual mesh filename=/home/rise/catkin_ws/src/stable_push_data_gen/assets/urdf/1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 scale=1 1 1

File: assets/urdf/1be987c137d37f0b7c15f7bdb6fa82dd_6/1be987c137d37f0b7c15f7bdb6fa82dd_6.urdf (robot description, URDF)
Before this commit: robot 1be987c137d37f0b7c15f7bdb6fa82dd_6, 1 links, 0 joints
Links:
- link 1be987c137d37f0b7c15f7bdb6fa82dd_6: geometry collision mesh filename=/home/rise/catkin_ws/src/stable_push_data_gen/assets/urdf/1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 scale=1 1 1; visual mesh filename=/home/rise/catkin_ws/src/stable_push_data_gen/assets/urdf/1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 scale=1 1 1

File: assets/urdf/1be987c137d37f0b7c15f7bdb6fa82dd_7/1be987c137d37f0b7c15f7bdb6fa82dd_7.urdf (robot description, URDF)
Before this commit: robot 1be987c137d37f0b7c15f7bdb6fa82dd_7, 1 links, 0 joints
Links:
- link 1be987c137d37f0b7c15f7bdb6fa82dd_7: geometry collision mesh filename=/home/rise/catkin_ws/src/stable_push_data_gen/assets/urdf/1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 scale=1 1 1; visual mesh filename=/home/rise/catkin_ws/src/stable_push_data_gen/assets/urdf/1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 scale=1 1 1

File: assets/urdf/1be987c137d37f0b7c15f7bdb6fa82dd_8/1be987c137d37f0b7c15f7bdb6fa82dd_8.urdf (robot description, URDF)
Before this commit: robot 1be987c137d37f0b7c15f7bdb6fa82dd_8, 1 links, 0 joints
Links:
- link 1be987c137d37f0b7c15f7bdb6fa82dd_8: geometry collision mesh filename=/home/rise/catkin_ws/src/stable_push_data_gen/assets/urdf/1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 scale=1 1 1; visual mesh filename=/home/rise/catkin_ws/src/stable_push_data_gen/assets/urdf/1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 scale=1 1 1

File: assets/urdf/1be987c137d37f0b7c15f7bdb6fa82dd_9/1be987c137d37f0b7c15f7bdb6fa82dd_9.urdf (robot description, URDF)
Before this commit: robot 1be987c137d37f0b7c15f7bdb6fa82dd_9, 1 links, 0 joints
Links:
- link 1be987c137d37f0b7c15f7bdb6fa82dd_9: geometry collision mesh filename=/home/rise/catkin_ws/src/stable_push_data_gen/assets/urdf/1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 scale=1 1 1; visual mesh filename=/home/rise/catkin_ws/src/stable_push_data_gen/assets/urdf/1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 scale=1 1 1

File: assets/urdf/2eb4cfc59205bb3a147c505998f546dd/2eb4cfc59205bb3a147c505998f546dd.urdf (robot description, URDF)
Before this commit: robot 2eb4cfc59205bb3a147c505998f546dd, 1 links, 0 joints
Links:
- link 2eb4cfc59205bb3a147c505998f546dd: geometry collision mesh filename=/home/rise/catkin_ws/src/stable_push_data_gen/assets/urdf/2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 scale=1 1 1; visual mesh filename=/home/rise/catkin_ws/src/stable_push_data_gen/assets/urdf/2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 scale=1 1 1

File: assets/urdf/2eb4cfc59205bb3a147c505998f546dd_0/2eb4cfc59205bb3a147c505998f546dd_0.urdf (robot description, URDF)
Before this commit: robot 2eb4cfc59205bb3a147c505998f546dd_0, 1 links, 0 joints
Links:
- link 2eb4cfc59205bb3a147c505998f546dd_0: geometry collision mesh filename=/home/rise/catkin_ws/src/stable_push_data_gen/assets/urdf/2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 scale=1 1 1; visual mesh filename=/home/rise/catkin_ws/src/stable_push_data_gen/assets/urdf/2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 scale=1 1 1

File: assets/urdf/2eb4cfc59205bb3a147c505998f546dd_1/2eb4cfc59205bb3a147c505998f546dd_1.urdf (robot description, URDF)
Before this commit: robot 2eb4cfc59205bb3a147c505998f546dd_1, 1 links, 0 joints
Links:
- link 2eb4cfc59205bb3a147c505998f546dd_1: geometry collision mesh filename=/home/rise/catkin_ws/src/stable_push_data_gen/assets/urdf/2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 scale=1 1 1; visual mesh filename=/home/rise/catkin_ws/src/stable_push_data_gen/assets/urdf/2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 scale=1 1 1

File: assets/urdf/2eb4cfc59205bb3a147c505998f546dd_2/2eb4cfc59205bb3a147c505998f546dd_2.urdf (robot description, URDF)
Before this commit: robot 2eb4cfc59205bb3a147c505998f546dd_2, 1 links, 0 joints
Links:
- link 2eb4cfc59205bb3a147c505998f546dd_2: geometry collision mesh filename=/home/rise/catkin_ws/src/stable_push_data_gen/assets/urdf/2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 scale=1 1 1; visual mesh filename=/home/rise/catkin_ws/src/stable_push_data_gen/assets/urdf/2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 scale=1 1 1

File: assets/urdf/2eb4cfc59205bb3a147c505998f546dd_3/2eb4cfc59205bb3a147c505998f546dd_3.urdf (robot description, URDF)
Before this commit: robot 2eb4cfc59205bb3a147c505998f546dd_3, 1 links, 0 joints
Links:
- link 2eb4cfc59205bb3a147c505998f546dd_3: geometry collision mesh filename=/home/rise/catkin_ws/src/stable_push_data_gen/assets/urdf/2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 scale=1 1 1; visual mesh filename=/home/rise/catkin_ws/src/stable_push_data_gen/assets/urdf/2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 scale=1 1 1

File: assets/urdf/2eb4cfc59205bb3a147c505998f546dd_4/2eb4cfc59205bb3a147c505998f546dd_4.urdf (robot description, URDF)
Before this commit: robot 2eb4cfc59205bb3a147c505998f546dd_4, 1 links, 0 joints
Links:
- link 2eb4cfc59205bb3a147c505998f546dd_4: geometry collision mesh filename=/home/rise/catkin_ws/src/stable_push_data_gen/assets/urdf/2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 scale=1 1 1; visual mesh filename=/home/rise/catkin_ws/src/stable_push_data_gen/assets/urdf/2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 scale=1 1 1

File: assets/urdf/2eb4cfc59205bb3a147c505998f546dd_5/2eb4cfc59205bb3a147c505998f546dd_5.urdf (robot description, URDF)
Before this commit: robot 2eb4cfc59205bb3a147c505998f546dd_5, 1 links, 0 joints
Links:
- link 2eb4cfc59205bb3a147c505998f546dd_5: geometry collision mesh filename=/home/rise/catkin_ws/src/stable_push_data_gen/assets/urdf/2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 scale=1 1 1; visual mesh filename=/home/rise/catkin_ws/src/stable_push_data_gen/assets/urdf/2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 scale=1 1 1

File: assets/urdf/2eb4cfc59205bb3a147c505998f546dd_6/2eb4cfc59205bb3a147c505998f546dd_6.urdf (robot description, URDF)
Before this commit: robot 2eb4cfc59205bb3a147c505998f546dd_6, 1 links, 0 joints
Links:
- link 2eb4cfc59205bb3a147c505998f546dd_6: geometry collision mesh filename=/home/rise/catkin_ws/src/stable_push_data_gen/assets/urdf/2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 scale=1 1 1; visual mesh filename=/home/rise/catkin_ws/src/stable_push_data_gen/assets/urdf/2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 scale=1 1 1

File: assets/urdf/2eb4cfc59205bb3a147c505998f546dd_7/2eb4cfc59205bb3a147c505998f546dd_7.urdf (robot description, URDF)
Before this commit: robot 2eb4cfc59205bb3a147c505998f546dd_7, 1 links, 0 joints
Links:
- link 2eb4cfc59205bb3a147c505998f546dd_7: geometry collision mesh filename=/home/rise/catkin_ws/src/stable_push_data_gen/assets/urdf/2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 scale=1 1 1; visual mesh filename=/home/rise/catkin_ws/src/stable_push_data_gen/assets/urdf/2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 scale=1 1 1
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