Commit message: ready to generate data from server

File: assets/pusher_urdf/pusher_vertical/pusher_vertical.urdf (robot description, URDF)
Before this commit: robot gripper, 7 links, 6 joints
Links:
- link eef: geometry visual box size=0.01 0.08 0.01
Joints:
- removed joint joint3
- added joint eef: type revolute, parent link2, child eef, axis 0 0 1, limit lower=-10 upper=10 effort=10 velocity=10
- joint joint4: axis 1 0 0 -> 0 1 0; limit lower=0.0 upper=0.04 effort=20 velocity=0.2 -> lower=-0.04 upper=0.04 effort=20 velocity=10; origin xyz=0 0.025 0.105 rpy=0 0 0 -> xyz=0 0.04 0.100 rpy=0 0 0; type fixed -> prismatic
- joint joint5: axis -1 0 0 -> 0 -1 0; limit lower=0.0 upper=0.04 effort=20 velocity=0.2 -> lower=-0.04 upper=0.04 effort=20 velocity=10; origin xyz=0 -0.025 0.105 rpy=0 0 0 -> xyz=0 -0.04 0.100 rpy=0 0 0; type fixed -> prismatic

Commit message: change gripper width

File: assets/pusher_urdf/pusher_vertical/pusher_vertical.urdf (robot description, URDF)
Before this commit: robot gripper, 7 links, 6 joints
Links:
- link eef: geometry 
