Commit message: hanyang gripper setting

File: assets/pusher_urdf/pusher.urdf (robot description, URDF)
Before this commit: robot gripper, 7 links, 6 joints
Links:
- removed link eef
- removed link left_finger
- removed link right_finger
- added link eef_p, mass 0.05
- added link eef_z, mass 0.05; visual box size=0.015 0.015 0.015
- link eef_y: mass None -> 0.05; geometry visual box size=0 0 0
Joints:
- removed joint eef
- removed joint joint4
- removed joint joint5
- added joint eef_p_joint: type revolute, parent eef_y, child eef_p, axis 0 1 0, limit lower=-10 upper=10 effort=100 velocity=100
- added joint eef_z_joint: type revolute, parent link2, child eef_z, axis 0 0 1, limit lower=-10 upper=10 effort=10 velocity=10
- joint eef_y_joint: axis 0 1 0 -> 1 0 0; limit lower=-10 upper=10 effort=100 velocity=100 -> lower=-0.1 upper=0.1 effort=10 velocity=10; origin (none) -> xyz=0 0 0 rpy=0 0 0; parent eef -> eef_z; type revolute -> prismatic
