Commit message: hanyang gripper setting - mesh dir name change from mesh to meshes

File: assets/pusher_urdf/hanyang/pusher.urdf (robot description, URDF)
Before this commit: robot pusher, 11 links, 10 joints
Links:
- link finger_1_1_link: geometry collision mesh filename=/home/jongsoo/catkin_ws/src/stable_push_data_gen/assets/pus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; visual mesh filename=/home/jongsoo/catkin_ws/src/stable_push_data_gen/assets/pus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
- link finger_1_2_link: geometry collision mesh filename=/home/jongsoo/catkin_ws/src/stable_push_data_gen/assets/pus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; visual mesh filename=/home/jongsoo/catkin_ws/src/stable_push_data_gen/assets/pus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
- link finger_2_1_link: geometry collision mesh filename=/home/jongsoo/catkin_ws/src/stable_push_data_gen/assets/pus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; visual mesh filename=/home/jongsoo/catkin_ws/src/stable_push_data_gen/assets/pus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
- link finger_2_2_link: geometry collision mesh filename=/home/jongsoo/catkin_ws/src/stable_push_data_gen/assets/pus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; visual mesh filename=/home/jongsoo/catkin_ws/src/stable_push_data_gen/assets/pus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

Commit message: hanyang gripper setting

File: assets/pusher_urdf/hanyang/pusher.urdf (robot description, URDF)
Before this commit: robot pusher, 11 links, 10 joints
Links:
- link finger_1_1_link: geometry collision mesh filename=/home/rise/catkin_ws/src/stable_push_data_gen/assets/pusher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; visual mesh filename=/home/rise/catkin_ws/src/stable_push_data_gen/assets/pusher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
- link finger_1_2_link: geometry collision mesh filename=/home/rise/catkin_ws/src/stable_push_data_gen/assets/pusher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; visual mesh filename=/home/rise/catkin_ws/src/stable_push_data_gen/assets/pusher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
- link finger_2_1_link: geometry collision mesh filename=/home/rise/catkin_ws/src/stable_push_data_gen/assets/pusher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; visual mesh filename=/home/rise/catkin_ws/src/stable_push_data_gen/assets/pusher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
- link finger_2_2_link: geometry collision mesh filename=/home/rise/catkin_ws/src/stable_push_data_gen/assets/pusher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; visual mesh filename=/home/rise/catkin_ws/src/stable_push_data_gen/assets/pusher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
Joints:
- joint eef_y_joint: limit lower=-0.1 upper=0.1 effort=10 velocity=10 -> lower=-0.1 upper=0 effort=10 velocity=10

File: assets/pusher_urdf/pusher.urdf (robot description, URDF)
Before this commit: robot gripper, 6 links, 5 joints
Joints:
- joint eef_y_joint: limit lower=-0.1 upper=0.1 effort=10 velocity=10 -> lower=0 upper=0.1 effort=10 velocity=10
